File: ecad/ecad.kicad_pcb (KiCad board)
At the start: 4 copper layers, 130.5 x 110 mm, 102 parts, among them J1 JTAG, J2 USB_C, J3 Display, Q1 SS8050, SW1 Kailh choc v2, SW10 RotaryEncoder_Switch, SW11 RotaryEncoder_Switch, SW12 Kailh choc v2, SW13 Kailh choc v2, SW14 Kailh choc v2, SW15 RESET, SW16 Kailh choc v2, SW17 Kailh choc v2, SW18 Kailh choc v2, SW19 Kailh choc v2, SW2 Kailh choc v2, SW20 Kailh choc v2, SW21 Kailh choc v2, SW22 Kailh choc v2, SW23 Kailh choc v2, SW24 Kailh choc v2, SW25 Kailh choc v2, SW3 Kailh choc v2, SW4 Kailh choc v2, SW5 Kailh choc v2, SW6 Kailh choc v2, SW7 Kailh choc v2, SW8 Kailh choc v2, SW9 Kailh choc v2, U1 AP2112K-3.3, U2 RP2040, U4 SN74LV1T34DBV, U5 W25Q128JVP, Y1 12MHz

Commit message: feat(ecad): general routing
Parts:
- removed Q1: SS8050, Package_TO_SOT_SMD:SOT-23
- added C19: 0.1u, Capacitor_SMD:C_0402_1005Metric, B.Cu at (171.4, 133.7)
- added C9: 4.7u, Capacitor_SMD:C_0402_1005Metric, B.Cu at (172.4, 133.7)
- added D41: WS2812B-2020, LED_SMD:LED_WS2812B-2020_PLCC4_2.0x2.0mm, B.Cu at (215.9, 108.8)
- added D42: WS2812B-2020, LED_SMD:LED_WS2812B-2020_PLCC4_2.0x2.0mm, B.Cu at (215.9, 112.3)
- added D43: WS2812B-2020, LED_SMD:LED_WS2812B-2020_PLCC4_2.0x2.0mm, B.Cu at (215.9, 115.8)
- added D44: WS2812B-2020, LED_SMD:LED_WS2812B-2020_PLCC4_2.0x2.0mm, B.Cu at (215.9, 119.4)
- added D45: WS2812B-2020, LED_SMD:LED_WS2812B-2020_PLCC4_2.0x2.0mm, B.Cu at (215.9, 123.0)
- added D46: WS2812B-2020, LED_SMD:LED_WS2812B-2020_PLCC4_2.0x2.0mm, B.Cu at (211.6, 108.8)
- added D47: WS2812B-2020, LED_SMD:LED_WS2812B-2020_PLCC4_2.0x2.0mm, B.Cu at (211.6, 112.3)
- added D48: WS2812B-2020, LED_SMD:LED_WS2812B-2020_PLCC4_2.0x2.0mm, B.Cu at (211.6, 115.8)
- added H5: MountingHole, MountingHole:MountingHole_2.2mm_M2_DIN965, F.Cu at (186.6, 100.2)
- added H6: MountingHole, MountingHole:MountingHole_2.2mm_M2_DIN965, F.Cu at (154.8, 100.2)
- added H7: MountingHole, MountingHole:MountingHole_2.2mm_M2_DIN965, F.Cu at (154.8, 147.6)
- added H8: MountingHole, MountingHole:MountingHole_2.2mm_M2_DIN965, F.Cu at (186.6, 147.6)
- added Q2: SS8050, Package_TO_SOT_SMD:SOT-23, B.Cu at (177.2, 134.1)
- added R11: 10, Resistor_SMD:R_0402_1005Metric, B.Cu at (174.4, 134.7)
- added R12: 1k, Resistor_SMD:R_0402_1005Metric, B.Cu at (179.8, 132.7)
- added R13: 10k, Resistor_SMD:R_0402_1005Metric, B.Cu at (173.4, 133.7)
- added kibuzzard-68D988DF: G***, kibuzzard-68D988DF, B.Cu at (154.4, 132.7)
- added kibuzzard-68D98929: G***, kibuzzard-68D98929, B.Cu at (153.1, 125.9)
- added kibuzzard-68D9895D: G***, kibuzzard-68D9895D, B.Cu at (161.2, 139.9)
- moved C18 124.2 mm to (177.1, 74.3), turned to 90 degrees
- moved U4 122.0 mm to (179.4, 74.0), turned to -90 degrees
- moved D32 120.2 mm to (181.3, 70.4), turned to 180 degrees
- moved R7 116.5 mm to (182.2, 76.2), turned to 0 degrees
- moved SW15 4.88 mm to (161.6, 132.7), turned to 180 degrees
- moved C1 4.71 mm to (164.3, 74.3)
- moved C2 3.90 mm to (162.0, 71.3), turned to 180 degrees
- moved C15 2.59 mm to (179.1, 125.0)
- moved Y1 1.88 mm to (176.4, 125.0)
- moved C14 0.93 mm to (171.3, 123.4)
- moved C4 0.93 mm to (172.3, 123.4)
- moved C16 0.92 mm to (173.7, 124.8), turned to -90 degrees
- moved R1 0.57 mm to (174.8, 122.6), turned to 0 degrees
- moved H1 0.50 mm to (190.7, 70.4)
- moved H2 0.50 mm to (66.2, 70.4)
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Connections:
- D17 pad 1: Net-(D13-DIN) -> Net-(D17-DOUT)
- D19 pad 1: Net-(D15-DIN) -> Net-(D19-DOUT)
- J3 pad 10: unconnected-(J3-Pin_10-Pad10) -> /DC
- J3 pad 11: unconnected-(J3-Pin_11-Pad11) -> /CS
- J3 pad 12: unconnected-(J3-Pin_12-Pad12) -> GND
- J3 pad 2: unconnected-(J3-Pin_2-Pad2) -> /LEDK
- J3 pad 3: unconnected-(J3-Pin_3-Pad3) -> +3.3V
- J3 pad 4: unconnected-(J3-Pin_4-Pad4) -> +3.3V
- J3 pad 5: unconnected-(J3-Pin_5-Pad5) -> +3.3V
- J3 pad 7: unconnected-(J3-Pin_7-Pad7) -> /RES
- J3 pad 8: unconnected-(J3-Pin_8-Pad8) -> /SDA
- J3 pad 9: unconnected-(J3-Pin_9-Pad9) -> /SCL
- SW24 pad 1: unconnected-(SW24-Pad1) -> Net-(U2-GPIO16)
- SW24 pad 2: unconnected-(SW24-Pad2) -> GND
- SW25 pad 1: unconnected-(SW25-Pad1) -> Net-(U2-GPIO17)
- SW25 pad 2: unconnected-(SW25-Pad2) -> GND
- U2 pad 12: unconnected-(U2-GPIO9-Pad12) -> /CS
- U2 pad 13: unconnected-(U2-GPIO10-Pad13) -> /SCL
- U2 pad 14: unconnected-(U2-GPIO11-Pad14) -> /SDA
- U2 pad 15: unconnected-(U2-GPIO12-Pad15) -> /BLK
- U2 pad 16: unconnected-(U2-GPIO13-Pad16) -> /RES
- U2 pad 17: unconnected-(U2-GPIO14-Pad17) -> /DC
- U2 pad 27: unconnected-(U2-GPIO16-Pad27) -> Net-(U2-GPIO16)
- U2 pad 28: unconnected-(U2-GPIO17-Pad28) -> Net-(U2-GPIO17)
- U2 pad 5: unconnected-(U2-GPIO3-Pad5) -> /Leds/DIN
Routing:
- net Net-(U2-GPIO16): track 0.00 -> 87.5 mm
- net Net-(U2-GPIO17): track 0.00 -> 69.6 mm
- net /Leds/DIN: track 0.00 -> 47.9 mm
- net /CS: track 0.00 -> 38.5 mm
- net /SCL: track 0.00 -> 36.0 mm
- net /SDA: track 0.00 -> 33.9 mm
- net GND: track 31.6 -> 64.2 mm, vias 34 -> 43
- net /DC: track 0.00 -> 31.0 mm
- net /RES: track 0.00 -> 29.9 mm
- net /BLK: track 0.00 -> 17.7 mm
- net Net-(U2-XIN): track 1.78 -> 11.4 mm
- net +5V: track 0.00 -> 8.41 mm
- net Net-(Q2-B): track 0.00 -> 6.43 mm
- net Net-(U4-A): track 0.00 -> 5.35 mm
- net Net-(D32-DIN): track 0.00 -> 4.67 mm
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- added copper zone on B.Cu, net +5V
Other:
- board size 130.5 x 110 mm -> 130.5 x 110.5 mm
