File: ecad/ecad.kicad_pcb (KiCad board)
At the start: 4 copper layers, 130.5 x 115 mm, 120 parts, among them J1 JTAG, J2 USB_C, J3 Display, Q2 SS8050, SW1 Kailh choc v2, SW10 RotaryEncoder_Switch, SW11 RotaryEncoder_Switch, SW12 Kailh choc v2, SW13 Kailh choc v2, SW14 Kailh choc v2, SW15 RESET, SW16 Kailh choc v2, SW17 Kailh choc v2, SW18 Kailh choc v2, SW19 Kailh choc v2, SW2 Kailh choc v2, SW20 Kailh choc v2, SW21 Kailh choc v2, SW22 Kailh choc v2, SW23 Kailh choc v2, SW24 Kailh choc v2, SW25 Kailh choc v2, SW3 Kailh choc v2, SW4 Kailh choc v2, SW5 Kailh choc v2, SW6 Kailh choc v2, SW7 Kailh choc v2, SW8 Kailh choc v2, SW9 Kailh choc v2, U1 AP2112K-3.3, U2 RP2040, U4 SN74LV1T34DBV, U5 W25Q128JVP, Y1 12MHz

Commit message: chore(ecad): update PCB layout, refresh STEP export and remove stale gerbers
Gerber files removed — to be regenerated from updated PCB.
New MCAD STEP export replaces ecad-export.step.
Parts:
- C1, C10, C11, C12, C13, C14, C15, C16, C17, C18, C19, C2, C3, C4, C5, C6, C7, C8, C9: footprint Capacitor_SMD:C_0402_1005Metric -> library:C_0402_1005Metric
- D1, D10, D11, D12, D2, D3, D33, D34, D35, D36, D37, D38, D39, D4, D40, D5, D6, D7, D8, D9: footprint Diode_SMD:D_SOD-123 -> library:D_SOD-123
- D13, D14, D17, D18, D19, D21, D22, D23, D25, D26, D27, D29, D30, D31, D32, D41, D42, D43, D45, D46, D47, D48: footprint LED_SMD:LED_WS2812B-2020_PLCC4_2.0x2.0mm -> library:LED_WS2812B-2020_PLCC4_2.0x2.0mm
- H1, H2, H3, H4: footprint sinhoo-smtso3030ctj:smtso3030ctj -> library:smtso3030ctj
- H10, H11, H12, H5: footprint MountingHole:MountingHole_3.2mm_M3_DIN965 -> library:MountingHole_3.2mm_M3_DIN965
- H6, H7, H8, H9: footprint MountingHole:MountingHole_2.2mm_M2_DIN965 -> library:MountingHole_2.2mm_M2_DIN965
- J1: footprint Connector_PinHeader_1.27mm:PinHeader_2x05_P1.27mm_Vertical_SMD -> library:PinHeader_2x05_P1.27mm_Vertical_SMD
- J2: footprint Connector_USB:USB_C_Receptacle_Amphenol_12401948E412A -> library:USB_C_Receptacle_Amphenol_12401948E412A
- J3: footprint Connector_FFC-FPC:Hirose_FH12-12S-0.5SH_1x12-1MP_P0.50mm_Horizontal -> library:Hirose_FH12-12S-0.5SH_1x12-1MP_P0.50mm_Horizontal
- Q2: footprint Package_TO_SOT_SMD:SOT-23 -> library:SOT-23
- R1: value 10k -> 0; footprint Resistor_SMD:R_0402_1005Metric -> library:R_0402_1005Metric
- R11, R12, R13, R2, R3, R7: footprint Resistor_SMD:R_0402_1005Metric -> library:R_0402_1005Metric
- R4: value 10k -> DNP; footprint Resistor_SMD:R_0402_1005Metric -> library:R_0402_1005Metric
- R5, R6: value 27,4 -> 5.1k; footprint Resistor_SMD:R_0402_1005Metric -> library:R_0402_1005Metric
- SW1, SW12, SW13, SW14, SW16, SW17, SW18, SW19, SW2, SW20, SW21, SW22, SW23, SW3, SW4, SW5, SW6, SW7, SW8, SW9: footprint PCM_Switch_Keyboard_Hotswap_Kailh:SW_Hotswap_Kailh_Choc_V2 -> library:SW_Hotswap_Kailh_Choc_V2
- SW10, SW11: footprint Rotary_Encoder:RotaryEncoder_Bourns_Vertical_PEC12R-3x17F-Sxxxx -> library:RotaryEncoder_Bourns_Vertical_PEC12R-3x17F-Sxxxx
- SW15: footprint Button_Switch_SMD:SW_Push_1P1T_NO_CK_KMR2 -> library:SW_Push_1P1T_NO_CK_KMR2
- SW24, SW25: value Kailh choc v2 -> ~; footprint Button_Switch_THT:SW_PUSH_6mm -> library:SW_PUSH_6mm
- U1, U4: footprint Package_TO_SOT_SMD:SOT-23-5 -> library:SOT-23-5
- U2: footprint Package_DFN_QFN:QFN-56-1EP_7x7mm_P0.4mm_EP3.2x3.2mm -> library:QFN-56-1EP_7x7mm_P0.4mm_EP3.2x3.2mm
- U5: footprint Package_SON:WSON-8-1EP_6x5mm_P1.27mm_EP3.4x4.3mm -> library:WSON-8-1EP_6x5mm_P1.27mm_EP3.4x4.3mm
- Y1: footprint Crystal:Crystal_SMD_Abracon_ABM8G-4Pin_3.2x2.5mm -> library:Crystal_SMD_Abracon_ABM8G-4Pin_3.2x2.5mm
- kibuzzard-68D988DF: footprint kibuzzard-68D988DF -> library:kibuzzard-68D988DF
- kibuzzard-68D98929: footprint kibuzzard-68D98929 -> library:kibuzzard-68D98929
- kibuzzard-68D9895D: footprint kibuzzard-68D9895D -> library:kibuzzard-68D9895D
